File: wombat.kicad_pcb (KiCad board)
At the start: 2 copper layers, 250.5 x 77.4 mm, 182 parts, among them J1 Conn_01x02, J2 Conn_01x03, SW1 SW_SPST, SW10 SW_SPST, SW101 SW_Push, SW11 SW_SPST, SW12 SW_SPST, SW13 SW_SPST, SW14 SW_SPST, SW15 SW_SPST, SW16 SW_SPST, SW17 SW_SPST, SW18 SW_SPST, SW19 SW_SPST, SW2 SW_SPST, SW20 SW_SPST, SW21 SW_SPST, SW22 SW_SPST, SW23 SW_SPST, SW24 SW_SPST, SW25 SW_SPST, SW26 SW_SPST, SW27 SW_SPST, SW28 SW_SPST, SW29 SW_SPST, SW3 SW_SPST, SW30 SW_SPST, SW31 SW_SPST, SW32 SW_SPST, SW33 SW_SPST, SW34 SW_SPST, SW35 SW_SPST, SW36 SW_SPST, SW37 SW_SPST, SW38 SW_SPST, SW39 SW_SPST, SW4 SW_SPST, SW40 SW_SPST, SW41 SW_SPST, SW42 SW_SPST, SW43 SW_SPST, SW44 SW_SPST, SW45 SW_SPST, SW46 SW_SPST, SW47 SW_SPST, SW48 SW_SPST, SW49 SW_SPST, SW5 SW_SPST, SW50 SW_SPST, SW51 SW_SPST, SW52 SW_SPST, SW6 SW_SPST, SW7 SW_SPST, SW8 SW_SPST, SW9 SW_SPST, U1 ProMicro

Commit message: Prep for routing
- North facing LEDs
- invert stabilizers
- New mounting holes (it's overkill, but i'd rather have options)
- implemented transitor to drive LEDs
- rename lib dir to wombat.pretty
- map pinouts for capslock and layer indicator LEDs
- implement breakaway tab with LED indicators
- reorient resistor placement
Parts:
- removed D133, D134, D135: LED, keebs-github:LED_D2.0mm_W4.8mm_H2.5mm_FlatTop_Reverse_Polarity
- removed H4: MountingHole_2.2mm_M2_DIN965_Pad, MountingHole:MountingHole_2.2mm_M2_DIN965_Pad
- removed J2: Conn_01x03, Connector_Wire:SolderWirePad_1x03_P3.81mm_Drill1.2mm
- removed R133, R134, R135: 300, Resistor_SMD:R_0805_2012Metric_Pad1.15x1.40mm_HandSolder
- added D151: LED, LED_SMD:LED_0805_2012Metric_Pad1.15x1.40mm_HandSolder, B.Cu at (21.0, 122.6)
- added D152: LED, LED_SMD:LED_0805_2012Metric_Pad1.15x1.40mm_HandSolder, B.Cu at (21.0, 127.6)
- added D153: LED, LED_SMD:LED_0805_2012Metric_Pad1.15x1.40mm_HandSolder, B.Cu at (21.0, 132.6)
- added D154: LED, wombat.pretty:LED_D2.0mm_W4.8mm_H2.5mm_FlatTop_Reverse_Polarity, B.Cu at (259.9, 66.9)
- added H10: MountingHole, wombat.pretty:MountingHole_2.2mm_M2_DIN965_Pad_Oval, F.Cu at (245.7, 132.3)
- added H101: Mouse_Bite, wombat.pretty:Mouse_Bite_04MM, F.Cu at (22.7, 120.3)
- added H102: Mouse_Bite, wombat.pretty:Mouse_Bite_04MM, F.Cu at (22.7, 124.7)
- added H103: Mouse_Bite, wombat.pretty:Mouse_Bite_04MM, F.Cu at (22.7, 129.1)
- added H104: Mouse_Bite, wombat.pretty:Mouse_Bite_04MM, F.Cu at (22.7, 133.5)
- added H11: MountingHole, wombat.pretty:MountingHole_2.2mm_M2_DIN965_Pad_Oval, F.Cu at (268.2, 101.3)
- added H12: MountingHole, wombat.pretty:MountingHole_2.2mm_M2_DIN965_Pad_Oval, F.Cu at (174.7, 68.4)
- added H9: MountingHole, wombat.pretty:MountingHole_2.2mm_M2_DIN965_Pad_Oval, F.Cu at (231.5, 68.4)
- added Q1: FDS6630A, Package_SO:SOIC-8_3.9x4.9mm_P1.27mm, F.Cu at (239.9, 118.7)
- added R1: 10K, Resistor_SMD:R_0805_2012Metric_Pad1.15x1.40mm_HandSolder, F.Cu at (239.8, 109.8)
- added R151: 300, Resistor_SMD:R_0805_2012Metric_Pad1.15x1.40mm_HandSolder, F.Cu at (24.9, 119.5)
- added R152: 300, Resistor_SMD:R_0805_2012Metric_Pad1.15x1.40mm_HandSolder, F.Cu at (24.9, 127.0)
- added R153: 300, Resistor_SMD:R_0805_2012Metric_Pad1.15x1.40mm_HandSolder, F.Cu at (24.9, 134.7)
- added R154: 300, wombat.pretty:R_0805_2012Metric_Pad1.15x1.40mm_HandSolder_Double_Sided, B.Cu at (254.6, 67.5)
- added R2: 100, Resistor_SMD:R_0805_2012Metric_Pad1.15x1.40mm_HandSolder, F.Cu at (243.4, 109.8)
- D101, D102, D103, D104, D105, D106, D107, D108, D109, D110, D111, D112, D113, D114, D115, D116, D117, D118, D119, D120, D121, D122, D123, D124, D125, D126, D127, D128, D129, D130, D131, D132: footprint keebs-github:LED_D2.0mm_W4.8mm_H2.5mm_FlatTop_Reverse_Polarity -> wombat.pretty:LED_D2.0mm_W4.8mm_H2.5mm_FlatTop_Reverse_Polarity
- H1, H3, H6, H7, H8: value MountingHole_2.2mm_M2_DIN965_Pad -> MountingHole; footprint MountingHole:MountingHole_2.2mm_M2_DIN965_Pad -> wombat.pretty:MountingHole_2.2mm_M2_DIN965_Pad_Oval
- H2, H5: value MountingHole_2.2mm_M2_DIN965_Pad_Oval -> MountingHole; footprint lib:MountingHole_2.2mm_M2_DIN965_Pad_Oval -> wombat.pretty:MountingHole_2.2mm_M2_DIN965_Pad_Oval
- J1: value Conn_01x02 -> Conn_01x05; footprint Connector_Wire:SolderWirePad_1x02_P3.81mm_Drill1.2mm -> Connector_PinSocket_2.00mm:PinSocket_1x05_P2.00mm_Vertical
- SW101: value SW_Push -> RESET
- SW30, SW34: footprint keebs-github:Mx_Alps_225 -> wombat.pretty:Mx_Alps_225_Inverted_Stabs
- moved J1 218.5 mm to (28.7, 87.3)
- moved H3 168.6 mm to (42.0, 68.4), turned to 90 degrees
- moved H6 75.8 mm to (117.8, 68.4), turned to 90 degrees
- moved H8 71.5 mm to (198.4, 132.3), turned to 90 degrees
- moved H2 71.4 mm to (44.1, 132.3), turned to 90 degrees
- moved H5 49.3 mm to (115.8, 132.3)
- moved H7 43.5 mm to (151.0, 98.0), turned to 90 degrees
- moved H1 27.4 mm to (24.3, 101.3)
- moved R128 18.5 mm to (145.7, 105.4), turned to 90 degrees
- moved R129 17.4 mm to (164.6, 105.4), turned to 90 degrees
- moved R127 14.9 mm to (126.7, 105.4), turned to 90 degrees
- moved R123 14.9 mm to (50.9, 105.4), turned to 90 degrees
- moved R124 14.9 mm to (69.9, 105.4), turned to 90 degrees
- moved R125 14.9 mm to (88.8, 105.4), turned to 90 degrees
- moved R126 14.9 mm to (107.8, 105.4), turned to 90 degrees
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Connections:
- D101 pad 1: GND -> Net-(D101-Pad1)
- D102 pad 1: GND -> Net-(D101-Pad1)
- D103 pad 1: GND -> Net-(D101-Pad1)
- D104 pad 1: GND -> Net-(D101-Pad1)
- D105 pad 1: GND -> Net-(D101-Pad1)
- D106 pad 1: GND -> Net-(D101-Pad1)
- D107 pad 1: GND -> Net-(D101-Pad1)
- D108 pad 1: GND -> Net-(D101-Pad1)
- D109 pad 1: GND -> Net-(D101-Pad1)
- D110 pad 1: GND -> Net-(D101-Pad1)
- D111 pad 1: GND -> Net-(D101-Pad1)
- D112 pad 1: GND -> Net-(D101-Pad1)
- D113 pad 1: GND -> Net-(D101-Pad1)
- D114 pad 1: GND -> Net-(D101-Pad1)
- D115 pad 1: GND -> Net-(D101-Pad1)
- D116 pad 1: GND -> Net-(D101-Pad1)
- D117 pad 1: GND -> Net-(D101-Pad1)
- D118 pad 1: GND -> Net-(D101-Pad1)
- D119 pad 1: GND -> Net-(D101-Pad1)
- D120 pad 1: GND -> Net-(D101-Pad1)
- D121 pad 1: GND -> Net-(D101-Pad1)
- D122 pad 1: GND -> Net-(D101-Pad1)
- D123 pad 1: GND -> Net-(D101-Pad1)
- D124 pad 1: GND -> Net-(D101-Pad1)
- D125 pad 1: GND -> Net-(D101-Pad1)
- D126 pad 1: GND -> Net-(D101-Pad1)
- D127 pad 1: GND -> Net-(D101-Pad1)
- D128 pad 1: GND -> Net-(D101-Pad1)
- D129 pad 1: GND -> Net-(D101-Pad1)
- D130 pad 1: GND -> Net-(D101-Pad1)
- D131 pad 1: GND -> Net-(D101-Pad1)
- D132 pad 1: GND -> Net-(D101-Pad1)
- J1 pad 1: +5V -> /LED_WASD
- J1 pad 2: GND -> /LED_CAPSLOCK
- R101 pad 1: Net-(D101-Pad2) -> +5V
- R101 pad 2: /BACKLIGHT_PWM -> Net-(D101-Pad2)
- R102 pad 1: Net-(D102-Pad2) -> +5V
- R102 pad 2: /BACKLIGHT_PWM -> Net-(D102-Pad2)
- R103 pad 1: Net-(D103-Pad2) -> +5V
- R103 pad 2: /BACKLIGHT_PWM -> Net-(D103-Pad2)
- R104 pad 1: Net-(D104-Pad2) -> +5V
- R104 pad 2: /BACKLIGHT_PWM -> Net-(D104-Pad2)
- R105 pad 1: Net-(D105-Pad2) -> +5V
- R105 pad 2: /BACKLIGHT_PWM -> Net-(D105-Pad2)
- R106 pad 1: Net-(D106-Pad2) -> +5V
- R106 pad 2: /BACKLIGHT_PWM -> Net-(D106-Pad2)
- R107 pad 1: Net-(D107-Pad2) -> +5V
- R107 pad 2: /BACKLIGHT_PWM -> Net-(D107-Pad2)
- R108 pad 1: Net-(D108-Pad2) -> +5V
- R108 pad 2: /BACKLIGHT_PWM -> Net-(D108-Pad2)
- R109 pad 1: Net-(D109-Pad2) -> +5V
- R109 pad 2: /BACKLIGHT_PWM -> Net-(D109-Pad2)
- R110 pad 1: Net-(D110-Pad2) -> +5V
- R110 pad 2: /BACKLIGHT_PWM -> Net-(D110-Pad2)
- R111 pad 1: Net-(D111-Pad2) -> +5V
- R111 pad 2: /BACKLIGHT_PWM -> Net-(D111-Pad2)
- R112 pad 1: Net-(D112-Pad2) -> +5V
- R112 pad 2: /BACKLIGHT_PWM -> Net-(D112-Pad2)
- R113 pad 1: Net-(D113-Pad2) -> +5V
- R113 pad 2: /BACKLIGHT_PWM -> Net-(D113-Pad2)
- R114 pad 1: Net-(D114-Pad2) -> +5V
- R114 pad 2: /BACKLIGHT_PWM -> Net-(D114-Pad2)
- R115 pad 1: Net-(D115-Pad2) -> +5V
- R115 pad 2: /BACKLIGHT_PWM -> Net-(D115-Pad2)
- R116 pad 1: Net-(D116-Pad2) -> +5V
- R116 pad 2: /BACKLIGHT_PWM -> Net-(D116-Pad2)
- R117 pad 1: Net-(D117-Pad2) -> +5V
- R117 pad 2: /BACKLIGHT_PWM -> Net-(D117-Pad2)
- R118 pad 1: Net-(D118-Pad2) -> +5V
- R118 pad 2: /BACKLIGHT_PWM -> Net-(D118-Pad2)
- R119 pad 1: Net-(D119-Pad2) -> +5V
- R119 pad 2: /BACKLIGHT_PWM -> Net-(D119-Pad2)
- R120 pad 1: Net-(D120-Pad2) -> +5V
- R120 pad 2: /BACKLIGHT_PWM -> Net-(D120-Pad2)
- R121 pad 1: Net-(D121-Pad2) -> +5V
- R121 pad 2: /BACKLIGHT_PWM -> Net-(D121-Pad2)
- R122 pad 1: Net-(D122-Pad2) -> +5V
- R122 pad 2: /BACKLIGHT_PWM -> Net-(D122-Pad2)
- R123 pad 1: Net-(D123-Pad2) -> +5V
- R123 pad 2: /BACKLIGHT_PWM -> Net-(D123-Pad2)
- R124 pad 1: Net-(D124-Pad2) -> +5V
- R124 pad 2: /BACKLIGHT_PWM -> Net-(D124-Pad2)
- R125 pad 1: Net-(D125-Pad2) -> +5V
- R125 pad 2: /BACKLIGHT_PWM -> Net-(D125-Pad2)
- R126 pad 1: Net-(D126-Pad2) -> +5V
- R126 pad 2: /BACKLIGHT_PWM -> Net-(D126-Pad2)
- R127 pad 1: Net-(D127-Pad2) -> +5V
- R127 pad 2: /BACKLIGHT_PWM -> Net-(D127-Pad2)
- R128 pad 1: Net-(D128-Pad2) -> +5V
- R128 pad 2: /BACKLIGHT_PWM -> Net-(D128-Pad2)
- R129 pad 1: Net-(D129-Pad2) -> +5V
- R129 pad 2: /BACKLIGHT_PWM -> Net-(D129-Pad2)
- R130 pad 1: Net-(D130-Pad2) -> +5V
- R130 pad 2: /BACKLIGHT_PWM -> Net-(D130-Pad2)
- R131 pad 1: Net-(D131-Pad2) -> +5V
- R131 pad 2: /BACKLIGHT_PWM -> Net-(D131-Pad2)
- R132 pad 1: Net-(D132-Pad2) -> +5V
- R132 pad 2: /BACKLIGHT_PWM -> Net-(D132-Pad2)
- SW101 pad 1: Net-(SW101-Pad1) -> GND
- SW101 pad 2: Net-(SW101-Pad2) -> /RESET
- U1 pad 22: Net-(SW101-Pad1) -> /RESET
- U1 pad 23: Net-(SW101-Pad2) -> GND
- U1 pad 3: GND -> Net-(U1-Pad3)
- U1 pad 4: GND -> Net-(U1-Pad3)
Routing:
- net /BACKLIGHT_PWM: track 696.2 -> 0.00 mm, vias 2 -> 0
- net /row_3: track 344.1 -> 0.00 mm, vias 1 -> 0
- net /col_4: track 283.4 -> 0.00 mm
- net /col_5: track 270.2 -> 0.00 mm
- net /row_2: track 262.8 -> 0.00 mm, vias 2 -> 0
- net /row_0: track 262.7 -> 0.00 mm
- net /col_1: track 260.5 -> 0.00 mm
- net /col_6: track 241.2 -> 0.00 mm, vias 1 -> 0
- net /row_1: track 241.1 -> 0.00 mm, vias 1 -> 0
- net /col_2: track 233.6 -> 0.00 mm
- net /col_3: track 217.7 -> 0.25 mm
- net /col_7: track 212.3 -> 0.00 mm, vias 1 -> 0
- net /col_8: track 181.0 -> 0.00 mm
- net /col_9: track 146.4 -> 0.17 mm
- net Net-(SW101-Pad2): track 133.9 -> 0.00 mm, vias 1 -> 0
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Other:
- board size 250.5 x 77.4 mm -> 253.5 x 77.4 mm
- net class Power: clearance 0.5 -> 0.2; trace_width 0.55 -> 0.4; via_dia 1.1 -> 0.9; via_drill 0.7 -> 0.6
- board text added: "CAPS"
- board text added: "L1"
- board text added: "L2"
- board text added: "L3"
- board text removed: "GND"
- board text removed: "LED A"
- board text removed: "LED B"
- board text removed: "LED C"
- board text removed: "VCC"
